File: digiport-general/digiport-general.kicad_sch (KiCad schematic)
At the start: 36 parts, among them J1 Audio&PTT, J2 USB/CIV/CAT, J3 USB_C_Receptacle_USB2.0_16P, U1 CH334P, U2 CM108B, U3 CH340X, U4 CH442E, Y1 12MHz

Commit message: digiport-gerneral bug fixed, update cable pinout document
Parts:
- removed JP2: FT891/Other, digiport:SolderJumper2-BCu, symbol Jumper:SolderJumper_2_Open
- removed JP4: YAESU/ICOM, Jumper:SolderJumper-3_P1.3mm_Bridged12_RoundedPad1.0x1.5mm, symbol Jumper:SolderJumper_3_Bridged12
- removed JP5: FSKK_EN, Jumper:SolderJumper-3_P1.3mm_Bridged12_RoundedPad1.0x1.5mm, symbol Jumper:SolderJumper_3_Bridged12
- added JP1b: FT891/Other, digiport:SolderJumper3-BCu, symbol Jumper:SolderJumper_3_Bridged12
- added JP2a: Yaesu/ICOM, digiport:SolderJumper-BCu-Bridged, symbol Jumper:SolderJumper_2_Bridged
- added JP3: FSKK_EN, digiport:SolderJumper2-BCu, symbol Jumper:SolderJumper_2_Open
- renumbered JP1 to JP1a, JP3 to JP2b, JP6 to JP4
Connections:
- net +5V: now also JP1b.1 (A)
- net PC_RxD: now also JP1b.3 (B)
- net PC_TxD: now also JP2a.1 (A)
- net RIGD_T: now also JP1b.2 (C)
- net RIG_AUOUT: now reaches C11.1, J1.T, JP4.2 (B), R6.2
- net GND/RIG_FSK renamed RIG_FSK
- net RIG_FSK: now also JP3.2 (B)
- net RIG_FSKK renamed PC_DTR
- net PC_DTR: now also JP3.1 (A)
- net RIG_PTT renamed PC_RTS
- net RIG_RX/GND renamed RIG_RX
- net RIG_RX: now also JP2a.2 (B)
Other:
- note added: "Jumper设置： 1、FT-891模式：JP1a断开、JP1b短接1-2（默认设置）。 2、FT-81x/8x7：JP1a短接、JP1b短接2-3， JP2a断开、JP2b短接（默认设置）。 3、ICOM模式：JP1a短接、JP1b短接2-3， JP2a短接，JP2b断开。 4、FSKK使能：JP3短接。 5、电台输出衰减：JP4断开。"
- note removed: "Jumper设置： 1、FT-891模式：JP1、JP2断开（默认设置）。 2、其他YAESU模式：JP1、JP2短接， JP3断开（默认设置）， JP4 1-2短接，2-3断开（默认设置）。 3、ICOM模式：JP1、JP2短接， JP3短接， JP4 1-2断开，2-3短接。 4、FSKK使能：JP5 1-2断开，2-3短接。 5、电台输出衰减：JP6断开。"
- moved on the sheet: C11, C12, R5
